Commit message: .

File: rbpodo_ros2/rbpodo_description/robots/rb10_1300e_u.urdf_new.xacro (robot description, xacro)
@@ -15,5 +15,5 @@
   <xacro:property name="wrist2_tc" value="${1}" />
   <xacro:property name="wrist3_tc" value="${1}" />
-  <xacro:rb_6dof model_id="rb10_1300e_u" prefix="$(arg prefix)" tcp_name="tcp" tcp_xyz="0.143832 -0.26 0.04234" tcp_rpy="0 -1.57079632679 3.14159265359" />
+  <xacro:rb_6dof model_id="rb10_1300e_u" prefix="$(arg prefix)" tcp_name="tcp" tcp_xyz="0.143832 -0.1447 0.04234" tcp_rpy="0 -1.57079632679 3.14159265359" />
   <xacro:rb_6dof_ros2_control prefix="$(arg prefix)" robot_ip="$(arg robot_ip)" cb_simulation="$(arg cb_simulation)" use_fake_hardware="$(arg use_fake_hardware)" fake_sensor_commands="$(arg fake_sensor_commands)" torque_constants="${[base_tc, shoulder_tc, elbow_tc, wrist1_tc, wrist2_tc, wrist3_tc]}" />
 </robot>

File: rbpodo_ros2/rbpodo_description/robots/rb10_1300e_u_new.urdf (robot description, URDF)
Before this commit: robot rb10_1300e_u, 8 links, 7 joints
Links:
- added link eoat, mass 4; collision mesh filename=package://rbpodo_description/meshes/rb10_1300e_u/collision/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; visual mesh filename=package://rbpodo_description/meshes/rb10_1300e_u/visual/eoa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
Joints:
- added joint eoat_joint: type fixed, parent link6, child eoat, origin xyz=0 -0.1153 0 rpy=0 0 0
- joint base: limit lower=-3.14 upper=3.14 effort=10 velocity=3.14 -> lower=-6.28 upper=6.28 effort=10 velocity=3.14
- joint elbow: limit lower=-3.14 upper=3.14 effort=10 velocity=3.14 -> lower=-2.87 upper=2.87 effort=10 velocity=3.14
- joint shoulder: limit lower=-3.14 upper=3.14 effort=10 velocity=3.14 -> lower=-6.28 upper=6.28 effort=10 velocity=3.14
- joint tcp_joint: origin xyz=0.143832 -0.26 0.04234 rpy=0 -1.57079632679 3.14159265359 -> xyz=0.143832 -0.1447 0.04234 rpy=0 -1.57079632679 3.14159265359; parent link6 -> eoat
- joint wrist1: limit lower=-3.14 upper=3.14 effort=10 velocity=3.14 -> lower=-6.28 upper=6.28 effort=10 velocity=3.14
- joint wrist2: limit lower=-3.14 upper=3.14 effort=10 velocity=3.14 -> lower=-6.28 upper=6.28 effort=10 velocity=3.14
- joint wrist3: limit lower=-3.14 upper=3.14 effort=10 velocity=3.14 -> lower=-6.28 upper=6.28 effort=10 velocity=3.14
